File: RemotePCB.kicad_sch (KiCad schematic)
At the start: 0 parts

Commit message: remote schematic
Parts:
- added 100 F: C, symbol Device:C
- added M1: HC-12, HC-12:MA05-1, symbol HC-12:HC-12
- added U1: ESP32-S3-WROOM-1U-N16R8, ESP32-S3-WROOM-1U-N16R8:XCVR_ESP32-S3-WROOM-1U-N16R8, symbol ESP32-S3-WROOM-1U-N16R8:ESP32-S3-WROOM-1U-N16R8
Connections:
- new net: 100 F.2, M1.1 (VCC), U1.2 (3V3)
- new net: M1.3 (RXD), U1.17 (IO9)
- new net: M1.4 (TXD), U1.18 (IO10)
- new net: M1.5 (SET), U1.4 (IO4)
- new net: M1.GND (GND1), M1.GND1
- new net GND: 100 F.1, M1.2 (GND), U1.1 (GND), U1.40 (GND), U1.41_1 (GND), U1.41_2 (GND), U1.41_3 (GND), U1.41_4 (GND), U1.41_5 (GND), U1.41_6 (GND), U1.41_7 (GND), U1.41_8 (GND), U1.41_9 (GND)
