File: RemotePCB.kicad_sch (KiCad schematic)
At the start: 0 parts

Commit message: Added initial symbols for the peripherals and controller
Parts:
- added C1: 220 mF, symbol Device:C_Polarized
- added M1: HC-12, HC-12:MA05-1, symbol HC-12:HC-12
- added OLEDScreen: SSD1306, symbol SSD1306-128x64_OLED:SSD1306
- added U1: ESP32-S3-WROOM-1U-N16R8, ESP32-S3-WROOM-1U-N16R8:XCVR_ESP32-S3-WROOM-1U-N16R8, symbol ESP32-S3-WROOM-1U-N16R8:ESP32-S3-WROOM-1U-N16R8
Connections:
- new net: C1.1, M1.1 (VCC)
- new net: C1.2, M1.2 (GND)
- new net: M1.GND (GND1), M1.GND1
- new net GND: U1.1 (GND), U1.40 (GND), U1.41_1 (GND), U1.41_2 (GND), U1.41_3 (GND), U1.41_4 (GND), U1.41_5 (GND), U1.41_6 (GND), U1.41_7 (GND), U1.41_8 (GND), U1.41_9 (GND)
